Commit message: added better notes for README, fixed urdf to work with teaching lab robots, made launch file for torque relay

File: springcontroller/flat_urdf_files/ceeorobot_flat.urdf (robot description, URDF)
Before this commit: robot ceeorobot, 15 links, 14 joints
Links:
- removed link ur3e_base
- removed link ur3e_base_link
- removed link ur3e_base_link_inertia
- removed link ur3e_flange
- removed link ur3e_forearm_link
- removed link ur3e_ft_frame
- removed link ur3e_shoulder_link
- removed link ur3e_tool0
- removed link ur3e_upper_arm_link
- removed link ur3e_wrist_1_link
- removed link ur3e_wrist_2_link
- removed link ur3e_wrist_3_link
- added link base
- added link base_link
- added link base_link_inertia, mass 2.0; collision mesh filename=file:///home/kat/workspace/src/ceeorobot_cell/ceeorobot_des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; visual mesh filename=file:///home/kat/workspace/src/ceeorobot_cell/ceeorobot_des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
- added link flange
- added link forearm_link, mass 1.26; collision mesh filename=file:///home/kat/workspace/src/ceeorobot_cell/ceeorobot_des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; visual mesh filename=file:///home/kat/workspace/src/ceeorobot_cell/ceeorobot_des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
- added link ft_frame
- added link shoulder_link, mass 2.0; collision mesh filename=file:///home/kat/workspace/src/ceeorobot_cell/ceeorobot_des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; visual mesh filename=file:///home/kat/workspace/src/ceeorobot_cell/ceeorobot_des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
- added link tool0
- added link upper_arm_link, mass 3.42; collision mesh filename=file:///home/kat/workspace/src/ceeorobot_cell/ceeorobot_des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; visual mesh filename=file:///home/kat/workspace/src/ceeorobot_cell/ceeorobot_des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
- added link wrist_1_link, mass 0.8; collision mesh filename=file:///home/kat/workspace/src/ceeorobot_cell/ceeorobot_des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; visual mesh filename=file:///home/kat/workspace/src/ceeorobot_cell/ceeorobot_des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
- added link wrist_2_link, mass 0.8; collision mesh filename=file:///home/kat/workspace/src/ceeorobot_cell/ceeorobot_des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; visual mesh filename=file:///home/kat/workspace/src/ceeorobot_cell/ceeorobot_des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
- added link wrist_3_link, mass 0.35; collision mesh filename=file:///home/kat/workspace/src/ceeorobot_cell/ceeorobot_des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; visual mesh filename=file:///home/kat/workspace/src/ceeorobot_cell/ceeorobot_des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
Joints:
- removed joint ur3e_base_joint
- removed joint ur3e_base_link-base_fixed_joint
- removed joint ur3e_base_link-base_link_inertia
- removed joint ur3e_elbow_joint
- removed joint ur3e_flange-tool0
- removed joint ur3e_shoulder_lift_joint
- removed joint ur3e_shoulder_pan_joint
- removed joint ur3e_wrist_1_joint
- removed joint ur3e_wrist_2_joint
- removed joint ur3e_wrist_3-flange
- removed joint ur3e_wrist_3_joint
- removed joint ur3e_wrist_3_link-ft_frame
- added joint base_joint: type fixed, parent robot_mount, child base_link, origin xyz=0 0 0 rpy=0 0 0
- added joint base_link-base_fixed_joint: type fixed, parent base_link, child base, origin xyz=0 0 0 rpy=0 0 3.141592653589793
- added joint base_link-base_link_inertia: type fixed, parent base_link, child base_link_inertia, origin xyz=0 0 0 rpy=0 0 3.141592653589793
- added joint elbow_joint: type revolute, parent upper_arm_link, child forearm_link, origin xyz=-0.24365 0 0 rpy=0 0 0, axis 0 0 1, limit lower=-3.141592653589793 upper=3.141592653589793 effort=28.0 velocity=3.141592653589793
- added joint flange-tool0: type fixed, parent flange, child tool0, origin xyz=0 0 0 rpy=1.5707963267948966 0 1.5707963267948966
- added joint shoulder_lift_joint: type revolute, parent shoulder_link, child upper_arm_link, origin xyz=0 0 0 rpy=1.570796327 0 0, axis 0 0 1, limit lower=-6.283185307179586 upper=6.283185307179586 effort=56.0 velocity=3.141592653589793
- added joint shoulder_pan_joint: type revolute, parent base_link_inertia, child shoulder_link, origin xyz=0 0 0.1519 rpy=0 0 0, axis 0 0 1, limit lower=-6.283185307179586 upper=6.283185307179586 effort=56.0 velocity=3.141592653589793
- added joint wrist_1_joint: type revolute, parent forearm_link, child wrist_1_link, origin xyz=-0.21325 0 0.11235 rpy=0 0 0, axis 0 0 1, limit lower=-6.283185307179586 upper=6.283185307179586 effort=12.0 velocity=6.283185307179586
- added joint wrist_2_joint: type revolute, parent wrist_1_link, child wrist_2_link, origin xyz=0 -0.08535 -1.750557762378351e-11 rpy=1.570796327 0 0, axis 0 0 1, limit lower=-6.283185307179586 upper=6.283185307179586 effort=12.0 velocity=6.283185307179586
- added joint wrist_3-flange: type fixed, parent wrist_3_link, child flange, origin xyz=0 0 0 rpy=0 -1.5707963267948966 -1.5707963267948966
- added joint wrist_3_joint: type continuous, parent wrist_2_link, child wrist_3_link, origin xyz=0 0.0819 -1.679797079540562e-11 rpy=1.570796326589793 3.141592653589793 3.141592653589793, axis 0 0 1, limit effort=12.0 velocity=6.283185307179586
- added joint wrist_3_link-ft_frame: type fixed, parent wrist_3_link, child ft_frame, origin xyz=0 0 0 rpy=3.141592653589793 0 0

Commit message: added different config file for demo

File: springcontroller/flat_urdf_files/ceeorobot_flat.urdf (robot description, URDF)
Before this commit: robot ceeorobot, 15 links, 14 joints
Links:
- removed link tool0
- added link tool0_controller
Joints:
- joint flange-tool0: child tool0 -> tool0_controller
