Commit message: Redefine world origin to table height at robot base center; eye-target y-offset to 20cm
world was only coincident with base_link's own origin because both flat
URDFs' base_joint had an identity (0,0,0) transform -- not a physical
necessity, just how the file happened to be authored. Mounting hardware
puts base_link 2cm above the real table, so base_joint's z origin is now
0.02 (x/y unchanged -- base_link's origin is already the mounting-bolt
center), putting world's origin at table height instead.

This makes gen3_collision_scene.yaml's earlier per-object -2cm offset
unnecessary; reverted the table/camera_tower poses back to their
flush-at-table-height values now that world itself starts there.

Both flat URDFs carry an xacro "do not hand-edit" banner; there's no
regeneration script in this repo, so these files are the actual runtime
source (see README's urdf_path default), but a future xacro re-export
would silently drop this hand edit.

Also corrects EYE_TARGET_Y_OFFSET_CM to 20cm (+5cm from the original
15cm, per follow-up correction -- not the earlier "set to 5cm" reading).

Co-Authored-By: Claude Sonnet 5 <noreply@anthropic.com>
Claude-Session: https://claude.ai/code/session_0179rJAqDCTMcF2fwdpLyKYp

File: springcontroller/flat_urdf_files/gen3_kinova_flat.urdf (robot description, URDF)
Before this commit: robot gen3, 19 links, 18 joints
Joints:
- joint base_joint: origin xyz=0 0 0 rpy=0 0 0 -> xyz=0 0 0.02 rpy=0 0 0

File: springcontroller/flat_urdf_files/gen3_kinova_flat_arm_only.urdf (robot description, URDF)
Before this commit: robot gen3, 11 links, 10 joints
Joints:
- joint base_joint: origin xyz=0 0 0 rpy=0 0 0 -> xyz=0 0 0.02 rpy=0 0 0
