Commit message: Vendor Gen2 URDF meshes; error loudly if the collision model fails
The ROS 1 description packages moved out of ~/sandbox/src (and won't
necessarily exist on a deployment machine), which silently broke
gen2_robotiq_flat.urdf: its absolute mesh paths went missing, and
URDFArmConfiguration only warnings.warn()s, so virtual_spring_node would
have run with no self-collision checking.

- Copy the 21 meshes the URDF uses (11 MB) into meshes/gen2_robotiq/ and
  install them; the URDF now references package://springcontroller/meshes/...
  like gen3_kinova_flat.urdf's package://kortex_description meshes.
- make_gen2_robotiq_urdf.sh: source dirs default to the new locations and
  are env-overridable; vendor_urdf_meshes.py fails if any mesh is missing.
- virtual_spring_node logs an ERROR when srdf_path is set but the collision
  model didn't load.

Verified offline: with an install-layout AMENT_PREFIX_PATH the URDF loads
with 17 collision geometries and 0 false collisions at candle; without it,
the collision model fails (now reported as an error). SRDF unchanged.

Co-Authored-By: Claude Opus 5.5 <noreply@anthropic.com>

File: springcontroller/flat_urdf_files/gen2_robotiq_flat.urdf (robot description, URDF)
Before this commit: robot j2s7s300_robotiq, 20 links, 19 joints
Links:
- link gripper_base_link: geometry collision mesh filename=package://springcontroller/meshes/gen2_robotiq/robotiq/mesh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; visual mesh filename=package://springcontroller/meshes/gen2_robotiq/robotiq/mesh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
- link gripper_finger1_finger_link: geometry collision mesh filename=package://springcontroller/meshes/gen2_robotiq/robotiq/mesh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; visual mesh filename=package://springcontroller/meshes/gen2_robotiq/robotiq/mesh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
- link gripper_finger1_finger_tip_link: geometry collision mesh filename=package://springcontroller/meshes/gen2_robotiq/robotiq/mesh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; visual mesh filename=package://springcontroller/meshes/gen2_robotiq/robotiq/mesh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
- link gripper_finger1_inner_knuckle_link: geometry collision mesh filename=package://springcontroller/meshes/gen2_robotiq/robotiq/mesh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; visual mesh filename=package://springcontroller/meshes/gen2_robotiq/robotiq/mesh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
- link gripper_finger1_knuckle_link: geometry collision mesh filename=package://springcontroller/meshes/gen2_robotiq/robotiq/mesh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; visual mesh filename=package://springcontroller/meshes/gen2_robotiq/robotiq/mesh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
- link gripper_finger2_finger_link: geometry collision mesh filename=package://springcontroller/meshes/gen2_robotiq/robotiq/mesh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; visual mesh filename=package://springcontroller/meshes/gen2_robotiq/robotiq/mesh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
- link gripper_finger2_finger_tip_link: geometry collision mesh filename=package://springcontroller/meshes/gen2_robotiq/robotiq/mesh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; visual mesh filename=package://springcontroller/meshes/gen2_robotiq/robotiq/mesh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
- link gripper_finger2_inner_knuckle_link: geometry collision mesh filename=package://springcontroller/meshes/gen2_robotiq/robotiq/mesh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; visual mesh filename=package://springcontroller/meshes/gen2_robotiq/robotiq/mesh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
- link gripper_finger2_knuckle_link: geometry collision mesh filename=package://springcontroller/meshes/gen2_robotiq/robotiq/mesh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; visual mesh filename=package://springcontroller/meshes/gen2_robotiq/robotiq/mesh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
- link j2s7s300_link_1: geometry collision mesh filename=package://springcontroller/meshes/gen2_robotiq/kinova/meshe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; visual mesh filename=package://springcontroller/meshes/gen2_robotiq/kinova/meshe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
- link j2s7s300_link_2: geometry collision mesh filename=package://springcontroller/meshes/gen2_robotiq/kinova/meshe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; visual mesh filename=package://springcontroller/meshes/gen2_robotiq/kinova/meshe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
- link j2s7s300_link_3: geometry collision mesh filename=package://springcontroller/meshes/gen2_robotiq/kinova/meshe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; visual mesh filename=package://springcontroller/meshes/gen2_robotiq/kinova/meshe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
- link j2s7s300_link_4: geometry collision mesh filename=package://springcontroller/meshes/gen2_robotiq/kinova/meshe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; visual mesh filename=package://springcontroller/meshes/gen2_robotiq/kinova/meshe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
- link j2s7s300_link_5: geometry collision mesh filename=package://springcontroller/meshes/gen2_robotiq/kinova/meshe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; visual mesh filename=package://springcontroller/meshes/gen2_robotiq/kinova/meshe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
- link j2s7s300_link_6: geometry collision mesh filename=package://springcontroller/meshes/gen2_robotiq/kinova/meshe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; visual mesh filename=package://springcontroller/meshes/gen2_robotiq/kinova/meshe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
- link j2s7s300_link_7: geometry collision mesh filename=package://springcontroller/meshes/gen2_robotiq/poli2/meshes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; visual mesh filename=package://springcontroller/meshes/gen2_robotiq/poli2/meshes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
- link j2s7s300_link_base: geometry collision mesh filename=package://springcontroller/meshes/gen2_robotiq/kinova/meshe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; visual mesh filename=package://springcontroller/meshes/gen2_robotiq/kinova/meshe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
